File: PCB/Power supply/Power supply/Power supply.kicad_pcb (KiCad board)
At the start: 2 copper layers, 160 x 120 mm, 121 parts, among them J1 Screw_Terminal_01x02, J10 Screw_Terminal_01x03, J11 Screw_Terminal_01x03, J12 Conn_01x02_Pin, J13 Conn_01x02_Pin, J14 Conn_01x02_Pin, J2 Screw_Terminal_01x03, J3 Screw_Terminal_01x02, J4 Conn_01x02_Pin, J5 Conn_01x02_Pin, J6 Conn_01x02_Pin, J7 Conn_01x02_Pin, J8 Screw_Terminal_01x03, J9 Screw_Terminal_01x03, Q1 BD140, Q2 BD139, Q3 IRF9540N, Q4 MMBT3904, Q5 MMBT3906, Q6 IRF540N, Q7 MMBT3904, Q8 MMBT3906, SW1 SW_DPST, SW2 SW_DPST, U1 LM393, U2 4001, U3 LM393, U4 4001, U5 L7812, U6 LM317_TO-220, U7 L7912, U8 LM337_TO220

Commit message: Minor changes to PCB design
Other:
- board text added: "Power supply board"
- board text removed: "Power amplifier -power supply board"
Changed lines of the file:
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@@
+	(gr_poly
+		(pts
+			(xy 198.012646 132.118488) (xy 197.974401 132.310756) (xy 197.899382 132.491868) (xy 197.790471 132.654864)
+			(xy 197.651854 132.793481) (xy 197.488858 132.902392) (xy 197.307746 132.977411) (xy 197.115478 133.015656)
+			(xy 196.919444 133.015656) (xy 196.727176 132.977411) (xy 196.546064 132.902392) (xy 196.383068 132.793481)
+			(xy 196.244451 132.654864) (xy 196.13554 132.491868) (xy 196.060521 132.310756) (xy 196.022276 132.118488)
+			(xy 196.017461 126.325471) (xy 196.022276 126.227454) (xy 196.060521 126.035186) (xy 196.13554 125.854074)
+			(xy 196.244451 125.691078) (xy 196.383068 125.552461) (xy 196.546064 125.44355) (xy 196.727176 125.368531)
+			(xy 196.919444 125.330286) (xy 197.115478 125.330286) (xy 197.307746 125.368531) (xy 197.488858 125.44355)
+			(xy 197.651854 125.552461) (xy 197.790471 125.691078) (xy 197.899382 125.854074) (xy 197.974401 126.035186)
+			(xy 198.012646 126.227454) (xy 198.017461 132.020471)
+		)
+		(stroke
+			(width 0.2)
+			(type solid)
+		)
+		(fill solid)
+		(layer "B.Mask")
+	)
 	(gr_poly
 		(pts
@@
 	(gr_poly
 		(pts
+			(xy 207.102276 126.307454) (xy 207.140521 126.115186) (xy 207.21554 125.934074) (xy 207.324451 125.771078)
+			(xy 207.463068 125.632461) (xy 207.626064 125.52355) (xy 207.807176 125.448531) (xy 207.999444 125.410286)
+			(xy 208.195478 125.410286) (xy 208.387746 125.448531) (xy 208.568858 125.52355) (xy 208.731854 125.632461)
+			(xy 208.870471 125.771078) (xy 208.979382 125.934074) (xy 209.054401 126.115186) (xy 209.092646 126.307454)
+			(xy 209.097461 132.005471) (xy 209.092646 132.103488) (xy 209.054401 132.295756) (xy 208.979382 132.476868)
+			(xy 208.870471 132.639864) (xy 208.731854 132.778481) (xy 208.568858 132.887392) (xy 208.387746 132.962411)
+			(xy 208.195478 133.000656) (xy 207.999444 133.000656) (xy 207.807176 132.962411) (xy 207.626064 132.887392)
+			(xy 207.463068 132.778481) (xy 207.324451 132.639864) (xy 207.21554 132.476868) (xy 207.140521 132.295756)
+			(xy 207.102276 132.103488) (xy 207.097461 126.405471)
+		)
+		(stroke
+			(width 0.2)
+			(type solid)
+		)
+		(fill solid)
+		(layer "B.Mask")
+	)
+	(gr_poly
+		(pts
 			(xy 140.695636 36.118177) (xy 140.903187 35.958916) (xy 141.129751 35.828111) (xy 141.371449 35.727997)
 			(xy 141.624147 35.660286) (xy 141.883521 35.626138) (xy 142.145134 35.626138) (xy 142.404509 35.660286)
@@
 	(gr_poly
 		(pts
+			(xy 195.512646 139.603488) (xy 195.474401 139.795756) (xy 195.399382 139.976868) (xy 195.290471 140.139864)
+			(xy 195.151854 140.278481) (xy 194.988858 140.387392) (xy 194.807746 140.462411) (xy 194.615478 140.500656)
+			(xy 194.419444 140.500656) (xy 194.227176 140.462411) (xy 194.046064 140.387392) (xy 193.883068 140.278481)
+			(xy 193.744451 140.139864) (xy 193.63554 139.976868) (xy 193.560521 139.795756) (xy 193.522276 139.603488)
+			(xy 193.517461 132.060471) (xy 193.522276 131.962454) (xy 193.560521 131.770186) (xy 193.63554 131.589074)
+			(xy 193.744451 131.426078) (xy 193.883068 131.287461) (xy 194.046064 131.17855) (xy 194.227176 131.103531)
+			(xy 194.419444 131.065286) (xy 194.615478 131.065286) (xy 194.807746 131.103531) (xy 194.988858 131.17855)
+			(xy 195.151854 131.287461) (xy 195.290471 131.426078) (xy 195.399382 131.589074) (xy 195.474401 131.770186)
+			(xy 195.512646 131.962454) (xy 195.517461 139.505471)
+		)
+		(stroke
+			(width 0.2)
+			(type solid)
+		)
+		(fill solid)
+		(layer "B.Mask")
+	)
+	(gr_poly
+		(pts
 			(xy 221.787338 57.079631) (xy 221.896249 57.242629) (xy 221.971268 57.423741) (xy 222.009512 57.616008)
 			(xy 222.009512 57.812042) (xy 221.971268 58.004309) (xy 221.896249 58.185421) (xy 221.787338 58.348418)
@@
 	(gr_poly
 		(pts
+			(xy 206.552646 139.723488) (xy 206.514401 139.915756) (xy 206.439382 140.096868) (xy 206.330471 140.259864)
+			(xy 206.191854 140.398481) (xy 206.028858 140.507392) (xy 205.847746 140.582411) (xy 205.655478 140.620656)
+			(xy 205.459444 140.620656) (xy 205.267176 140.582411) (xy 205.086064 140.507392) (xy 204.923068 140.398481)
+			(xy 204.784451 140.259864) (xy 204.67554 140.096868) (xy 204.600521 139.915756) (xy 204.562276 139.723488)
+			(xy 204.557461 132.005471) (xy 204.562276 131.907454) (xy 204.600521 131.715186) (xy 204.67554 131.534074)
+			(xy 204.784451 131.371078) (xy 204.923068 131.232461) (xy 205.086064 131.12355) (xy 205.267176 131.048531)
+			(xy 205.459444 131.010286) (xy 205.655478 131.010286) (xy 205.847746 131.048531) (xy 206.028858 131.12355)
+			(xy 206.191854 131.232461) (xy 206.330471 131.371078) (xy 206.439382 131.534074) (xy 206.514401 131.715186)
+			(xy 206.552646 131.907454) (xy 206.557461 139.625471)
+		)
+		(stroke
+			(width 0.2)
+			(type solid)
+		)
+		(fill solid)
+		(layer "B.Mask")
+	)
+	(gr_poly
+		(pts
 			(xy 203.112345 62.92884) (xy 203.304613 62.967085) (xy 203.485725 63.042104) (xy 203.648721 63.151015)
 			(xy 203.787338 63.289632) (xy 203.896249 63.452628) (xy 203.971268 63.63374) (xy 204.009513 63.826008)
@@
 		)
 	)
-	(gr_text "Power amplifier\n-power supply board"
-		(at 99 130 0)
-		(layer "F.SilkS")
-		(effects
-			(font
-				(size 3 2)
-				(thickness 0.3)
+	(gr_text "Power supply board"
+		(at 92 34 270)
+		(layer "F.SilkS")
+		(effects
+			(font
+				(size 4 2.5)
+				(thickness 0.4)
+				(bold yes)
 			)
 			(justify left)
