File: PCB/Power supply/Power supply/Power supply.kicad_pcb (KiCad board)
At the start: 2 copper layers, 160 x 120 mm, 121 parts, among them J1 Screw_Terminal_01x02, J10 Screw_Terminal_01x03, J11 Screw_Terminal_01x03, J12 Conn_01x02_Pin, J13 Conn_01x02_Pin, J14 Conn_01x02_Pin, J2 Screw_Terminal_01x03, J3 Screw_Terminal_01x02, J4 Conn_01x02_Pin, J5 Conn_01x02_Pin, J6 Conn_01x02_Pin, J7 Conn_01x02_Pin, J8 Screw_Terminal_01x03, J9 Screw_Terminal_01x03, Q1 BD140, Q2 BD139, Q3 IRF9540N, Q4 MMBT3904, Q5 MMBT3906, Q6 IRF540N, Q7 MMBT3904, Q8 MMBT3906, SW1 SW_DPST, SW2 SW_DPST, U1 LM393, U2 4001, U3 LM393, U4 4001, U5 L7812, U6 LM317_TO-220, U7 L7912, U8 LM337_TO220

Commit message: Did some simulations, fixed some mistakes in PSU schematic
Parts:
- R4, R7: value 1K -> 470R
- RV3, RV4: value 470R -> 330R
Connections:
- Q4 pad 1: OVERCURRENT_P -> Net-(Q4-B)
- Q5 pad 1: OVERCURRENT_N -> Net-(Q5-B)
- R18 pad 2: OVERCURRENT_P -> Net-(Q4-B)
- R22 pad 2: /Over-current/S_N -> S_N
- R24 pad 2: /Over-current/S_N -> S_N
- R26 pad 2: OVERCURRENT_N -> Net-(Q5-B)
- U2 pad 10: Net-(U2-Pad10) -> OVERCURRENT_P
- U2 pad 12: Net-(U2-Pad10) -> OVERCURRENT_P
- U2 pad 13: Net-(U2-Pad10) -> OVERCURRENT_P
- U3 pad 1: /Over-current/S_N -> S_N
- U4 pad 1: RESET_N -> S_N
- U4 pad 10: Net-(U4-Pad10) -> OVERCURRENT_N
- U4 pad 12: Net-(U4-Pad10) -> OVERCURRENT_N
- U4 pad 13: Net-(U4-Pad10) -> OVERCURRENT_N
- U4 pad 6: /Over-current/S_N -> RESET_N
Routing:
- net RESET_N: track 107.3 -> 132.9 mm
- net /Over-current/S_N: track 25.6 -> 0.00 mm
- net Net-(U4-Pad10): track 6.98 -> 0.00 mm
- net OVERCURRENT_N: track 86.7 -> 93.7 mm
- net OVERCURRENT_P: track 76.8 -> 83.7 mm
- net Net-(U2-Pad10): track 6.83 -> 0.00 mm
