File: PCB/Power supply/Power supply/IO.kicad_sch (KiCad schematic)
At the start: 30 parts, among them J10 Screw_Terminal_01x03, J11 Screw_Terminal_01x03, J12 Conn_01x02_Pin, J13 Conn_01x02_Pin, J14 Conn_01x02_Pin, J4 Conn_01x02_Pin, J5 Conn_01x02_Pin, J6 Conn_01x02_Pin, J7 Conn_01x02_Pin, J8 Screw_Terminal_01x03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

Commit message: Made Power Supply schematic prettier
Other:
- note added: "NPN B"
- note added: "NPN C"
- note added: "NPN E"
- note added: "PNP B"
- note added: "PNP C"
- note added: "PNP E"
- note removed: "NPN_B"
- note removed: "NPN_C"
- note removed: "NPN_E"
- note removed: "PNP_B"
- note removed: "PNP_C"
- note removed: "PNP_E"
Changed lines of the file:
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@@
 	(text "OVERCURRENT LED\nNEGATIVE RAIL\n"
 		(exclude_from_sim no)
-		(at 199.898 117.856 0)
+		(at 208.788 138.684 0)
 		(effects
 			(font
+				(face "AIGDT")
 				(size 2 2)
 				(thickness 0.6)
@@
 		(effects
 			(font
+				(face "AIGDT")
 				(size 2 2)
 				(thickness 0.6)
@@
 		)
 	)
-	(text "NPN_C\n"
+	(text "NPN C\n"
 		(exclude_from_sim no)
 		(at 25.4 53.34 0)
 		(effects
 			(font
+				(face "AIGDT")
 				(size 1 1)
 				(thickness 0.6)
@@
 	(text "PNP PASS TRANSISTOR\n(TIP36C)"
 		(exclude_from_sim no)
-		(at 48.514 20.574 0)
+		(at 46.99 20.066 0)
 		(effects
 			(font
+				(face "AIGDT")
 				(size 2 2)
 				(thickness 0.6)
@@
 		(effects
 			(font
+				(face "AIGDT")
 				(size 2 2)
 				(thickness 0.6)
@@
 		(effects
 			(font
+				(face "AIGDT")
 				(size 2 2)
 				(thickness 0.6)
@@
 		)
 	)
-	(text "PNP_C\n"
+	(text "PNP C\n"
 		(exclude_from_sim no)
-		(at 24.384 29.718 0)
+		(at 24.384 30.988 0)
 		(effects
 			(font
+				(face "AIGDT")
 				(size 1 1)
 				(thickness 0.6)
@@
 	(text "POWER LED\nNEGATIVE RAIL\n"
 		(exclude_from_sim no)
-		(at 136.144 118.364 0)
+		(at 135.89 122.428 0)
 		(effects
 			(font
+				(face "AIGDT")
 				(size 2 2)
 				(thickness 0.6)
@@
 		(effects
 			(font
+				(face "AIGDT")
 				(size 2 2)
 				(thickness 0.6)
@@
 	(text "POWER LED\nPOSITIVE RAIL\n"
 		(exclude_from_sim no)
-		(at 137.16 77.724 0)
+		(at 135.636 77.47 0)
 		(effects
 			(font
+				(face "AIGDT")
 				(size 2 2)
 				(thickness 0.6)
@@
 		(effects
 			(font
+				(face "AIGDT")
 				(size 2 2)
 				(thickness 0.6)
@@
 	(text "NPN PASS TRANSISTOR\n(TIP35C)"
 		(exclude_from_sim no)
-		(at 48.514 43.434 0)
+		(at 45.974 43.942 0)
 		(effects
 			(font
+				(face "AIGDT")
 				(size 2 2)
 				(thickness 0.6)
@@
 		(effects
 			(font
+				(face "AIGDT")
 				(size 2 2)
 				(thickness 0.6)
@@
 		)
 	)
-	(text "PNP_E\n"
+	(text "PNP E\n"
 		(exclude_from_sim no)
-		(at 24.638 33.02 0)
+		(at 24.638 34.29 0)
 		(effects
 			(font
+				(face "AIGDT")
 				(size 1 1)
 				(thickness 0.6)
@@
 		)
 	)
-	(text "PNP_B\n"
+	(text "PNP B\n"
 		(exclude_from_sim no)
-		(at 24.384 26.67 0)
+		(at 24.384 27.94 0)
 		(effects
 			(font
+				(face "AIGDT")
 				(size 1 1)
 				(thickness 0.6)
@@
 	(text "OVERCURRENT LED\nPOSITIVE RAIL\n"
 		(exclude_from_sim no)
-		(at 200.66 98.552 0)
+		(at 207.772 75.438 0)
 		(effects
 			(font
+				(face "AIGDT")
 				(size 2 2)
 				(thickness 0.6)
@@
 		(effects
 			(font
+				(face "AIGDT")
 				(size 2 2)
 				(thickness 0.6)
@@
 		)
 	)
-	(text "NPN_E\n"
+	(text "NPN E\n"
 		(exclude_from_sim no)
 		(at 25.654 56.642 0)
 		(effects
 			(font
+				(face "AIGDT")
 				(size 1 1)
 				(thickness 0.6)
@@
 		)
 	)
-	(text "NPN_B\n"
+	(text "NPN B\n"
 		(exclude_from_sim no)
 		(at 25.4 50.292 0)
 		(effects
 			(font
+				(face "AIGDT")
 				(size 1 1)
 				(thickness 0.6)
@@
 		(dnp no)
 		(property "Reference" "J5"
-			(at 241.3 34.2901 0)
+			(at 240.792 33.274 0)
 			(effects
 				(font
@@
 				)
 				(justify right)
+				(hide yes)
 			)
 		)
@@
 		(on_board yes)
 		(dnp no)
-		(fields_autoplaced yes)
 		(property "Reference" "J8"
-			(at 55.88 29.2099 0)
+			(at 51.562 25.146 0)
 			(effects
 				(font
@@
 				)
 				(justify left)
+				(hide yes)
 			)
 		)
@@
 				)
 				(justify right)
+				(hide yes)
 			)
 		)
@@
 		(on_board yes)
 		(dnp no)
-		(fields_autoplaced yes)
 		(property "Reference" "J6"
-			(at 173.99 33.0199 0)
+			(at 173.482 34.29 0)
 			(effects
 				(font
@@
 				)
 				(justify right)
+				(hide yes)
 			)
 		)
@@
 		(on_board yes)
 		(dnp no)
-		(fields_autoplaced yes)
 		(property "Reference" "J9"
-			(at 107.95 31.7499 0)
+			(at 104.14 27.686 0)
 			(effects
 				(font
@@
 		(dnp no)
 		(property "Reference" "J14"
-			(at 139.7 111.7601 0)
+			(at 139.446 110.49 0)
 			(effects
 				(font
@@
 				)
 				(justify right)
+				(hide yes)
 			)
 		)
@@
 		(dnp no)
 		(property "Reference" "J4"
-			(at 208.28 34.2901 0)
+			(at 208.026 33.274 0)
 			(effects
 				(font
@@
 				)
 				(justify right)
+				(hide yes)
 			)
 		)
@@
 		(on_board yes)
 		(dnp no)
-		(fields_autoplaced yes)
 		(property "Reference" "J10"
-			(at 138.43 33.0199 0)
+			(at 134.366 28.956 0)
 			(effects
 				(font
@@
 		(dnp no)
 		(property "Reference" "J13"
-			(at 139.7 87.6301 0)
+			(at 139.192 86.36 0)
 			(effects
 				(font
@@
 				)
 				(justify right)
+				(hide yes)
 			)
 		)
@@
 		(dnp no)
 		(property "Reference" "J11"
-			(at 55.88 54.6101 0)
+			(at 51.562 48.006 0)
 			(effects
 				(font
@@
 				)
 				(justify left)
+				(hide yes)
 			)
 		)
@@
 				)
 				(justify right)
+				(hide yes)
 			)
 		)
