File: PCB/Power supply/Power supply/Rectifier.sch.kicad_sch (KiCad schematic)
At the start: 23 parts, among them J1 Screw_Terminal_01x02, J2 Screw_Terminal_01x03, J3 Screw_Terminal_01x02, U1 LM393, U2 4001, U3 LM393, U4 4001

Commit message: Made Power Supply schematic prettier
Other:
- note removed: "RECTIFIER"
- moved on the sheet: C1, C2, C3, C4, D1, D2, D3, D4, J1, J2, J3, TP1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
