File: PCB/Amplifier/Amplifier/Amplifier.kicad_sch (KiCad schematic)
At the start: 0 parts

Commit message: Big commit after a long time :)
Other:
- added sheet Block diagram (block_diagram.kicad_sch)
- added sheet IO (io.kicad_sch)
Changed lines of the file:
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@@
 	)
 	(sheet
-		(at 63.5 50.8)
+		(at 66.04 57.15)
 		(size 40.64 25.4)
 		(fields_autoplaced yes)
@@
 		)
 		(property "Sheetname" "Invert stage"
-			(at 63.5 50.0884 0)
+			(at 66.04 56.4384 0)
 			(effects
 				(font
@@
 		)
 		(property "Sheetfile" "invert_stage.kicad_sch"
-			(at 63.5 76.7846 0)
+			(at 66.04 83.1346 0)
+			(effects
+				(font
+					(size 1.27 1.27)
+				)
+				(justify left top)
+			)
+		)
+		(instances
+			(project "Amplifier"
+				(path "/c90a190d-425c-4649-b2e7-4df291106ff4"
+					(page "5")
+				)
+			)
+		)
+	)
+	(sheet
+		(at 113.03 57.15)
+		(size 38.1 25.4)
+		(stroke
+			(width 0.1524)
+			(type solid)
+		)
+		(fill
+			(color 0 0 0 0.0000)
+		)
+		(property "Sheetname" "Gain stage"
+			(at 113.03 56.388 0)
+			(effects
+				(font
+					(size 1.27 1.27)
+				)
+				(justify left bottom)
+			)
+		)
+		(property "Sheetfile" "gain_stage.kicad_sch"
+			(at 113.03 83.1346 0)
+			(effects
+				(font
+					(size 1.27 1.27)
+				)
+				(justify left top)
+			)
+		)
+		(instances
+			(project "Amplifier"
+				(path "/c90a190d-425c-4649-b2e7-4df291106ff4"
+					(page "6")
+				)
+			)
+		)
+	)
+	(sheet
+		(at 19.05 57.15)
+		(size 40.64 25.4)
+		(fields_autoplaced yes)
+		(stroke
+			(width 0.1524)
+			(type solid)
+		)
+		(fill
+			(color 0 0 0 0.0000)
+		)
+		(property "Sheetname" "Input stage"
+			(at 19.05 56.4384 0)
+			(effects
+				(font
+					(size 1.27 1.27)
+				)
+				(justify left bottom)
+			)
+		)
+		(property "Sheetfile" "input_stage.kicad_sch"
+			(at 19.05 83.1346 0)
+			(effects
+				(font
+					(size 1.27 1.27)
+				)
+				(justify left top)
+			)
+		)
+		(instances
+			(project "Amplifier"
+				(path "/c90a190d-425c-4649-b2e7-4df291106ff4"
+					(page "4")
+				)
+			)
+		)
+	)
+	(sheet
+		(at 19.05 24.13)
+		(size 40.64 25.4)
+		(fields_autoplaced yes)
+		(stroke
+			(width 0.1524)
+			(type solid)
+		)
+		(fill
+			(color 0 0 0 0.0000)
+		)
+		(property "Sheetname" "Block diagram"
+			(at 19.05 23.4184 0)
+			(effects
+				(font
+					(size 1.27 1.27)
+				)
+				(justify left bottom)
+			)
+		)
+		(property "Sheetfile" "block_diagram.kicad_sch"
+			(at 19.05 50.1146 0)
+			(effects
+				(font
+					(size 1.27 1.27)
+				)
+				(justify left top)
+			)
+		)
+		(instances
+			(project "Amplifier"
+				(path "/c90a190d-425c-4649-b2e7-4df291106ff4"
+					(page "2")
+				)
+			)
+		)
+	)
+	(sheet
+		(at 66.04 24.13)
+		(size 40.64 25.4)
+		(fields_autoplaced yes)
+		(stroke
+			(width 0.1524)
+			(type solid)
+		)
+		(fill
+			(color 0 0 0 0.0000)
+		)
+		(property "Sheetname" "Power"
+			(at 66.04 23.4184 0)
+			(effects
+				(font
+					(size 1.27 1.27)
+				)
+				(justify left bottom)
+			)
+		)
+		(property "Sheetfile" "power.kicad_sch"
+			(at 66.04 50.1146 0)
 			(effects
 				(font
@@
 	)
 	(sheet
-		(at 17.78 50.8)
+		(at 158.75 57.15)
 		(size 38.1 25.4)
-		(stroke
-			(width 0.1524)
-			(type solid)
-		)
-		(fill
-			(color 0 0 0 0.0000)
-		)
-		(property "Sheetname" "Gain stage"
-			(at 17.78 50.038 0)
-			(effects
-				(font
-					(size 1.27 1.27)
-				)
-				(justify left bottom)
-			)
-		)
-		(property "Sheetfile" "gain_stage.kicad_sch"
-			(at 17.78 76.7846 0)
-			(effects
-				(font
-					(size 1.27 1.27)
-				)
-				(justify left top)
-			)
-		)
-		(instances
-			(project "Amplifier"
-				(path "/c90a190d-425c-4649-b2e7-4df291106ff4"
-					(page "4")
-				)
-			)
-		)
-	)
-	(sheet
-		(at 111.76 17.78)
-		(size 40.64 25.4)
-		(fields_autoplaced yes)
-		(stroke
-			(width 0.1524)
-			(type solid)
-		)
-		(fill
-			(color 0 0 0 0.0000)
-		)
-		(property "Sheetname" "Input stage"
-			(at 111.76 17.0684 0)
-			(effects
-				(font
-					(size 1.27 1.27)
-				)
-				(justify left bottom)
-			)
-		)
-		(property "Sheetfile" "input_stage.kicad_sch"
-			(at 111.76 43.7646 0)
-			(effects
-				(font
-					(size 1.27 1.27)
-				)
-				(justify left top)
-			)
-		)
-		(instances
-			(project "Amplifier"
-				(path "/c90a190d-425c-4649-b2e7-4df291106ff4"
-					(page "2")
-				)
-			)
-		)
-	)
-	(sheet
-		(at 63.5 17.78)
-		(size 40.64 25.4)
-		(fields_autoplaced yes)
-		(stroke
-			(width 0.1524)
-			(type solid)
-		)
-		(fill
-			(color 0 0 0 0.0000)
-		)
-		(property "Sheetname" "Power"
-			(at 63.5 17.0684 0)
-			(effects
-				(font
-					(size 1.27 1.27)
-				)
-				(justify left bottom)
-			)
-		)
-		(property "Sheetfile" "power.kicad_sch"
-			(at 63.5 43.7646 0)
-			(effects
-				(font
-					(size 1.27 1.27)
-				)
-				(justify left top)
-			)
-		)
-		(instances
-			(project "Amplifier"
-				(path "/c90a190d-425c-4649-b2e7-4df291106ff4"
-					(page "1")
-				)
-			)
-		)
-	)
-	(sheet
-		(at 17.78 17.78)
+		(fields_autoplaced yes)
+		(stroke
+			(width 0.1524)
+			(type solid)
+		)
+		(fill
+			(color 0 0 0 0.0000)
+		)
+		(property "Sheetname" "Output stage"
+			(at 158.75 56.4384 0)
+			(effects
+				(font
+					(size 1.27 1.27)
+				)
+				(justify left bottom)
+			)
+		)
+		(property "Sheetfile" "output_stage.kicad_sch"
+			(at 158.75 83.1346 0)
+			(effects
+				(font
+					(size 1.27 1.27)
+				)
+				(justify left top)
+			)
+		)
+		(instances
+			(project "Amplifier"
+				(path "/c90a190d-425c-4649-b2e7-4df291106ff4"
+					(page "7")
+				)
+			)
+		)
+	)
+	(sheet
+		(at 113.03 24.13)
 		(size 38.1 25.4)
 		(fields_autoplaced yes)
@@
 			(color 0 0 0 0.0000)
 		)
-		(property "Sheetname" "Output stage"
-			(at 17.78 17.0684 0)
-			(effects
-				(font
-					(size 1.27 1.27)
-				)
-				(justify left bottom)
-			)
-		)
-		(property "Sheetfile" "output_stage.kicad_sch"
-			(at 17.78 43.7646 0)
-			(effects
-				(font
-					(size 1.27 1.27)
-				)
-				(justify left top)
-			)
-		)
-		(instances
-			(project "Amplifier"
-				(path "/c90a190d-425c-4649-b2e7-4df291106ff4"
-					(page "5")
-				)
-			)
+		(property "Sheetname" "IO"
+			(at 113.03 23.4184 0)
+			(effects
+				(font
+					(size 1.27 1.27)
+				)
+				(justify left bottom)
+			)
+		)
+		(property "Sheetfile" "io.kicad_sch"
+			(at 113.03 50.1146 0)
+			(effects
+				(font
+					(size 1.27 1.27)
+				)
+				(justify left top)
+			)
+		)
+		(instances
+			(project "Amplifier"
+				(path "/c90a190d-425c-4649-b2e7-4df291106ff4"
+					(page "8")
+				)
+			)
