File: PCB/Amplifier/Amplifier/gain_stage.kicad_sch (KiCad schematic)
At the start: 12 parts, among them IC3 OPA1692IDR, K2 Relay_SPDT, Q12 NPN

Commit message: Worked on "amplifier" schematic
Parts:
- removed K2: Relay_SPDT, symbol Relay:Relay_SPDT
- added C24, C25: C, symbol Device:C
- added J3: SR5-3V-200-1C, SR53V2001C, symbol SamacSys_Parts:SR5-3V-200-1C
- added R34: 100, symbol Device:R
- added R47: 10k, symbol Device:R
- added TP10, TP11, TP12: TestPoint, symbol Connector:TestPoint
- R42: value 1k -> 10k
- R43: value 10k -> 100k
- R44: value R -> 150
- R45: value R -> 10k
Connections:
- net GAIN_INPUT: now also R34.1, TP10.1; no longer R40.1, R42.2
- net GND: now also R47.1
- net IN: now also J3.COM
- net X1: now also C24.2, J3.NO, TP11.1
- net X10: now also C25.2, J3.NC, TP12.1
- net at D9.2 (A), Q12.1 (C): now also J3.A1
- net at IC3.6 (-), R42.1, R43.2: now also C25.1
- net at IC3.2 (-), R40.2, R41.2: now also C24.1
- net GAIN_SELECT: now reaches R45.1
- net GAIN_SELECT: now also R47.2
- net at D9.1 (K), R44.2: now also J3.A2
- new net: R34.2, R40.1, R42.2
Other:
- title: (none) -> Gain stage
- moved on the sheet: Q12, R45

Commit message: Worked on amplifier schematic
Parts:
- IC3: footprint SOIC127P600X175-8N -> (none)
- J3: footprint SR53V2001C -> (none)
Changed lines of the file:
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@@
 			)
 		)
-		(property "Footprint" "SOIC127P600X175-8N"
+		(property "Footprint" ""
 			(at 143.51 -36.5 0)
 			(effects
@@
 			)
 		)
-		(property "Footprint" "SOIC127P600X175-8N"
+		(property "Footprint" ""
 			(at 144.78 13.03 0)
 			(effects
@@
 			)
 		)
-		(property "Footprint" "SOIC127P600X175-8N"
+		(property "Footprint" ""
 			(at 77.47 252.4 0)
 			(effects
@@
 			)
 		)
-		(property "Footprint" "SR53V2001C"
+		(property "Footprint" ""
 			(at 160.02 -30.15 0)
 			(effects

Commit message: Big commit after a long time :)
Parts:
- removed Q12: NPN, symbol Simulation_SPICE:NPN
- added C21: 100n, Capacitor_THT:C_Disc_D4.3mm_W1.9mm_P5.00mm, symbol Device:C
- added Q2: 2N3904, Package_TO_SOT_THT:TO-92_Inline, symbol Transistor_BJT:2N3904
- added RV1, RV2: 100, Potentiometer_THT:Potentiometer_Bourns_3296W_Vertical, symbol Device:R_Potentiometer_Trim
- C19: renamed from C24; value C -> 10p; footprint (none) -> Capacitor_THT:C_Disc_D4.3mm_W1.9mm_P5.00mm
- C20: renamed from C25; value C -> 10p; footprint (none) -> Capacitor_THT:C_Disc_D4.3mm_W1.9mm_P5.00mm
- C22: renamed from C21; footprint (none) -> Capacitor_THT:C_Disc_D4.3mm_W1.9mm_P5.00mm
- C23: renamed from C22; footprint (none) -> Capacitor_THT:C_Disc_D4.3mm_W1.9mm_P5.00mm
- D10: renamed from D9; value D -> 1N4007; footprint (none) -> Diode_THT:D_DO-15_P10.16mm_Horizontal
- K2: renamed from J3; footprint (none) -> SamacSys_Parts:SR53V2001C
- R20: renamed from R41; footprint (none) -> Resistor_THT:R_Axial_DIN0207_L6.3mm_D2.5mm_P10.16mm_Horizontal
- R21: renamed from R44; footprint (none) -> Resistor_THT:R_Axial_DIN0207_L6.3mm_D2.5mm_P10.16mm_Horizontal
- R22: renamed from R40; footprint (none) -> Resistor_THT:R_Axial_DIN0207_L6.3mm_D2.5mm_P10.16mm_Horizontal
- R23: renamed from R34; value 100 -> 47; footprint (none) -> Resistor_THT:R_Axial_DIN0207_L6.3mm_D2.5mm_P10.16mm_Horizontal
- R24: renamed from R43; footprint (none) -> Resistor_THT:R_Axial_DIN0207_L6.3mm_D2.5mm_P10.16mm_Horizontal
- R25: renamed from R45; footprint (none) -> Resistor_THT:R_Axial_DIN0207_L6.3mm_D2.5mm_P10.16mm_Horizontal
- R26: renamed from R42; footprint (none) -> Resistor_THT:R_Axial_DIN0207_L6.3mm_D2.5mm_P10.16mm_Horizontal
- R27: renamed from R47; footprint (none) -> Resistor_THT:R_Axial_DIN0207_L6.3mm_D2.5mm_P10.16mm_Horizontal
- TP10: renamed from TP11; footprint (none) -> Connector_Pin:Pin_D1.2mm_L11.3mm_W3.0mm_Flat
- TP11: renamed from TP10; footprint (none) -> Connector_Pin:Pin_D1.2mm_L11.3mm_W3.0mm_Flat
- TP12: footprint (none) -> Connector_Pin:Pin_D1.2mm_L11.3mm_W3.0mm_Flat
- U5: renamed from IC3; footprint (none) -> SamacSys_Parts:SOIC127P600X175-8N
Connections:
- net GAIN_SELECT: now also C21.1
- net GND: now also C21.2, Q2.1 (E)
- net X1: now also RV1.2, RV1.3; no longer R20.1
- net X10: now also RV2.2, RV2.3; no longer R24.1
- net at D10.2 (A), K2.A1: now also Q2.3 (C)
- net at R25.2: now also Q2.2 (B)
- new net: R24.1, RV2.1
- new net: R20.1, RV1.1
Other:
- moved on the sheet: D10, K2, R20, R21, R24, R25, R27, TP10, TP12
