File: PCB/Amplifier/Amplifier/input_stage.kicad_sch (KiCad schematic)
At the start: 19 parts, among them IC1 OPA1692IDR, J2 Conn_Coaxial

Commit message: Worked on "amplifier" schematic
Parts:
- removed R34: 100, symbol Device:R
- added TP5, TP6, TP7: TestPoint, symbol Connector:TestPoint
Connections:
- net INVERT_INPUT: now also C16.2, IC1.6 (-), IC1.7, TP7.1
- net at C14.2, IC1.1, R30.2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: now also TP6.1
- net at D5.2 (A), D6.1 (K), IC1.3 (+)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: now also TP5.1
Other:
- moved on the sheet: C15, C16, IC1B, R31, R32

Commit message: Worked on amplifier schematic
Parts:
- IC1: footprint SOIC127P600X175-8N -> (none)
Changed lines of the file:
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@@
 			)
 		)
-		(property "Footprint" "SOIC127P600X175-8N"
+		(property "Footprint" ""
 			(at 168.91 153.34 0)
 			(effects
@@
 			)
 		)
-		(property "Footprint" "SOIC127P600X175-8N"
+		(property "Footprint" ""
 			(at 100.33 234.62 0)
 			(effects
@@
 			)
 		)
-		(property "Footprint" "SOIC127P600X175-8N"
+		(property "Footprint" ""
 			(at 234.95 155.88 0)
 			(effects

Commit message: Big commit after a long time :)
Parts:
- removed R27: 100, symbol Device:R
- added C9: 1n, Capacitor_THT:C_Rect_L7.2mm_W2.5mm_P5.00mm_FKS2_FKP2_MKS2_MKP2, symbol Device:C
- added D4, D6: 1N4007, Diode_THT:D_DO-15_P10.16mm_Horizontal, symbol Device:D
- added R6: 47, Resistor_THT:R_Axial_DIN0207_L6.3mm_D2.5mm_P10.16mm_Horizontal, symbol Device:R
- C10: renamed from C16; value C -> 1n; footprint (none) -> Capacitor_THT:C_Rect_L7.2mm_W2.5mm_P5.00mm_FKS2_FKP2_MKS2_MKP2
- C11: renamed from C15; value C -> 1n; footprint (none) -> Capacitor_THT:C_Rect_L7.2mm_W2.5mm_P5.00mm_FKS2_FKP2_MKS2_MKP2
- C12: renamed from C14; value C -> 100n; footprint (none) -> Capacitor_THT:C_Disc_D4.3mm_W1.9mm_P5.00mm
- C13: renamed from C17; footprint (none) -> Capacitor_THT:C_Disc_D4.3mm_W1.9mm_P5.00mm
- C14: renamed from C18; footprint (none) -> Capacitor_THT:C_Disc_D4.3mm_W1.9mm_P5.00mm
- D3: renamed from D4; value D_Zener -> 8.2V; footprint (none) -> Diode_THT:D_DO-35_SOD27_P10.16mm_Horizontal
- D5: value D -> 1N4007; footprint (none) -> Diode_THT:D_DO-15_P10.16mm_Horizontal
- D7: renamed from D6; value D -> 1N4007; footprint (none) -> Diode_THT:D_DO-15_P10.16mm_Horizontal
- D8: renamed from D7; value D_Zener -> 8.2V; footprint (none) -> Diode_THT:D_DO-35_SOD27_P10.16mm_Horizontal
- J2: footprint (none) -> SamacSys_Parts:52220061
- R10: renamed from R29; footprint (none) -> Resistor_THT:R_Axial_DIN0207_L6.3mm_D2.5mm_P10.16mm_Horizontal
- R11: renamed from R30; value 100 -> 47; footprint (none) -> Resistor_THT:R_Axial_DIN0207_L6.3mm_D2.5mm_P10.16mm_Horizontal
- R5: renamed from R26; footprint (none) -> Resistor_THT:R_Axial_DIN0207_L6.3mm_D2.5mm_P10.16mm_Horizontal
- R7: renamed from R31; value R -> 560; footprint (none) -> Resistor_THT:R_Axial_DIN0207_L6.3mm_D2.5mm_P10.16mm_Horizontal
- R8: renamed from R32; value R -> 560; footprint (none) -> Resistor_THT:R_Axial_DIN0207_L6.3mm_D2.5mm_P10.16mm_Horizontal
- R9: renamed from R28; footprint (none) -> Resistor_THT:R_Axial_DIN0207_L6.3mm_D2.5mm_P10.16mm_Horizontal
- TP5: renamed from TP7; footprint (none) -> Connector_Pin:Pin_D1.2mm_L11.3mm_W3.0mm_Flat
- TP6: renamed from TP5; footprint (none) -> Connector_Pin:Pin_D1.2mm_L11.3mm_W3.0mm_Flat
- TP7: renamed from TP6; footprint (none) -> Connector_Pin:Pin_D1.2mm_L11.3mm_W3.0mm_Flat
- U3: renamed from IC1; footprint (none) -> SamacSys_Parts:SOIC127P600X175-8N
Connections:
- net +12V: now also D4.1 (K)
- net -12V: now also D6.2 (A)
- net INPUT: now also R6.1
- net INVERT_INPUT: now also C9.2
- net at C10.1, R7.2, R8.1: now also C9.1
- net at D5.2 (A), D7.1 (K), R9.1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: now also D4.2 (A), D6.1 (K), R6.2
Other:
- note added: "5 V_{rms} max."
- note added: "Buffer"
- note added: "Input protection, clamps to 9V peak"
- note added: "Sallen-Key, butterworth 200kHz"
- title: (none) -> Input stage
- moved on the sheet: C10, C11, C12, D3, D5, D7, D8, J2, R10, R11, R5, R7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
