File: PCB/Amplifier/Amplifier/invert_stage.kicad_sch (KiCad schematic)
At the start: 12 parts, among them IC2 OPA1692IDR, K1 Relay_SPDT, Q11 NPN

Commit message: Worked on "amplifier" schematic
Parts:
- removed K1: Relay_SPDT, symbol Relay:Relay_SPDT
- added J4: SR5-3V-200-1C, SR53V2001C, symbol SamacSys_Parts:SR5-3V-200-1C
- added R46: 10k, symbol Device:R
- added R48: 100, symbol Device:R
- added TP8, TP9: TestPoint, symbol Connector:TestPoint
- R35, R36, R37: value 1K -> 10k
- R38: value R -> 150
- R39: value R -> 10k
Connections:
- net GAIN_INPUT: now also J4.COM
- net GND: now also R46.1
- net INVERT: now also R46.2
- net INVERTED: now also J4.NO, TP8.1
- net INVERT_INPUT: now also R48.1; no longer IC2.3 (+), R35.1
- net NORMAL: now also J4.NC, TP9.1
- net at D8.2 (A), Q11.1 (C): now also J4.A1
- net at D8.1 (K), R38.2: now also J4.A2
- new net: IC2.3 (+), R35.1, R48.2
Other:
- moved on the sheet: D8, IC2A, IC2B, Q11, R33, R35, R36, R37, R38, R39

Commit message: Worked on amplifier schematic
Parts:
- IC2: footprint SOIC127P600X175-8N -> (none)
- J4: footprint SR53V2001C -> (none)
Changed lines of the file:
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@@
 			)
 		)
-		(property "Footprint" "SOIC127P600X175-8N"
+		(property "Footprint" ""
 			(at 154.94 7.95 0)
 			(effects
@@
 			)
 		)
-		(property "Footprint" "SR53V2001C"
+		(property "Footprint" ""
 			(at 195.58 -36.5 0)
 			(effects
@@
 			)
 		)
-		(property "Footprint" "SOIC127P600X175-8N"
+		(property "Footprint" ""
 			(at 154.94 139.37 0)
 			(effects
@@
 			)
 		)
-		(property "Footprint" "SOIC127P600X175-8N"
+		(property "Footprint" ""
 			(at 78.74 253.67 0)
 			(effects

Commit message: Big commit after a long time :)
Parts:
- removed Q11: NPN, symbol Simulation_SPICE:NPN
- added C15: 10p, Capacitor_THT:C_Disc_D4.3mm_W1.9mm_P5.00mm, symbol Device:C
- added C16: 100n, Capacitor_THT:C_Disc_D4.3mm_W1.9mm_P5.00mm, symbol Device:C
- added Q1: 2N3904, Package_TO_SOT_THT:TO-92_Inline, symbol Transistor_BJT:2N3904
- C17: renamed from C19; footprint (none) -> Capacitor_THT:C_Disc_D4.3mm_W1.9mm_P5.00mm
- C18: renamed from C20; footprint (none) -> Capacitor_THT:C_Disc_D4.3mm_W1.9mm_P5.00mm
- D9: renamed from D8; value D -> 1N4007; footprint (none) -> Diode_THT:D_DO-15_P10.16mm_Horizontal
- K1: renamed from J4; footprint (none) -> SamacSys_Parts:SR53V2001C
- R12: renamed from R38; footprint (none) -> Resistor_THT:R_Axial_DIN0207_L6.3mm_D2.5mm_P10.16mm_Horizontal
- R13: renamed from R33; value 100 -> 47; footprint (none) -> Resistor_THT:R_Axial_DIN0207_L6.3mm_D2.5mm_P10.16mm_Horizontal
- R14: renamed from R48; value 100 -> 47; footprint (none) -> Resistor_THT:R_Axial_DIN0207_L6.3mm_D2.5mm_P10.16mm_Horizontal
- R15: renamed from R39; footprint (none) -> Resistor_THT:R_Axial_DIN0207_L6.3mm_D2.5mm_P10.16mm_Horizontal
- R16: renamed from R36; footprint (none) -> Resistor_THT:R_Axial_DIN0207_L6.3mm_D2.5mm_P10.16mm_Horizontal
- R17: renamed from R46; footprint (none) -> Resistor_THT:R_Axial_DIN0207_L6.3mm_D2.5mm_P10.16mm_Horizontal
- R18: renamed from R35; footprint (none) -> Resistor_THT:R_Axial_DIN0207_L6.3mm_D2.5mm_P10.16mm_Horizontal
- R19: renamed from R37; footprint (none) -> Resistor_THT:R_Axial_DIN0207_L6.3mm_D2.5mm_P10.16mm_Horizontal
- TP8, TP9: footprint (none) -> Connector_Pin:Pin_D1.2mm_L11.3mm_W3.0mm_Flat
- U4: renamed from IC2; footprint (none) -> SamacSys_Parts:SOIC127P600X175-8N
Connections:
- net GND: now also C16.2, Q1.1 (E)
- net INVERT: now also C16.1
- net NORMAL: now also C15.2
- net at R16.1, R18.2, U4.6 (-): now also C15.1
- net at R15.2: now also Q1.2 (B)
- net at D9.2 (A), K1.A1: now also Q1.3 (C)
Other:
- title: (none) -> Invert stage
