File: PCB/Amplifier/Amplifier/output_stage.kicad_sch (KiCad schematic)
At the start: 41 parts, among them Q1 BD139, Q10 TIP2955G, Q2 BD140, Q3 BD140, Q4 BD139, Q5 BD139, Q6 BD139, Q7 BD139, Q8 BD140, Q9 TIP3055G, U1 OPA552U

Commit message: Worked on "amplifier" schematic
Parts:
- added R49: 1Meg, symbol Device:R
- added TP13, TP14: TestPoint, symbol Connector:TestPoint
- R3, R6: value 22K -> 10k
Connections:
- net GND: now also R49.2
- net IN: now also R49.1, TP13.1
- net OUTPUT: now also TP14.1
Other:
- title: (none) -> Output stage
- moved on the sheet: R19, RV2

Commit message: Worked on amplifier schematic
Parts:
- added R50: R, symbol Device:R
- added RV3: R_Potentiometer_Trim, symbol Device:R_Potentiometer_Trim
- R15, R16: value 0.1 -> 0.1 2W
- R17: value 900 -> 900 2W
- R49: value 1Meg -> R
Connections:
- net GND: now also R50.2; no longer R49.2
- net IN: no longer TP13.1, U1.3 (+)
- new net: R49.2, RV3.1
- new net: R50.1, RV3.2, RV3.3, TP13.1, U1.3 (+)
Other:
- moved on the sheet: C1, C2, C23, C3, D1, JP1, JP2, Q1, Q10, Q2, Q3, Q4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

Commit message: Big commit after a long time :)
Parts:
- removed JP1: ~, Jumper:SolderJumper-2_P1.3mm_Bridged2Bar_Pad1.0x1.5mm, symbol Jumper:SolderJumper_2_Bridged
- removed JP2: SolderJumper_2_Bridged, Jumper:SolderJumper-2_P1.3mm_Bridged2Bar_Pad1.0x1.5mm, symbol Jumper:SolderJumper_2_Bridged
- added C24, C31: 100n, Capacitor_THT:C_Disc_D4.3mm_W1.9mm_P5.00mm, symbol Device:C
- added C26, C32: 1u, Capacitor_THT:C_Rect_L7.2mm_W4.5mm_P5.00mm_FKS2_FKP2_MKS2_MKP2, symbol Device:C
- added C30: DNP, Capacitor_THT:C_Disc_D4.3mm_W1.9mm_P5.00mm, symbol Device:C
- added C34: 100p, Capacitor_THT:C_Disc_D4.3mm_W1.9mm_P5.00mm, symbol Device:C
- added D11, D12: 1N4007, Diode_THT:D_DO-15_P10.16mm_Horizontal, symbol Device:D
- added J14: Conn_01x02_Pin, Connector_JST:JST_XH_B2B-XH-A_1x02_P2.50mm_Vertical, symbol Connector:Conn_01x02_Pin
- added J3: NPN1, TerminalBlock_Phoenix:TerminalBlock_Phoenix_MKDS-1,5-3_1x03_P5.00mm_Horizontal, symbol Connector:Screw_Terminal_01x03
- added J4: NPN2, TerminalBlock_Phoenix:TerminalBlock_Phoenix_MKDS-1,5-3_1x03_P5.00mm_Horizontal, symbol Connector:Screw_Terminal_01x03
- added J5: NPN3, TerminalBlock_Phoenix:TerminalBlock_Phoenix_MKDS-1,5-3_1x03_P5.00mm_Horizontal, symbol Connector:Screw_Terminal_01x03
- added J6: PNP2, TerminalBlock_Phoenix:TerminalBlock_Phoenix_MKDS-1,5-3_1x03_P5.00mm_Horizontal, symbol Connector:Screw_Terminal_01x03
- added J7: PNP1, TerminalBlock_Phoenix:TerminalBlock_Phoenix_MKDS-1,5-3_1x03_P5.00mm_Horizontal, symbol Connector:Screw_Terminal_01x03
- added J8: Conn_01x03_Pin, Connector_JST:JST_XH_B3B-XH-A_1x03_P2.50mm_Vertical, symbol Connector:Conn_01x03_Pin
- added R42: DNP, Resistor_THT:R_Axial_DIN0207_L6.3mm_D2.5mm_P10.16mm_Horizontal, symbol Device:R
- added R45: 0R, Resistor_THT:R_Axial_DIN0207_L6.3mm_D2.5mm_P10.16mm_Horizontal, symbol Device:R
- added R53: 150k, Resistor_THT:R_Axial_DIN0207_L6.3mm_D2.5mm_P10.16mm_Horizontal, symbol Device:R
- C25: renamed from C2; footprint (none) -> Capacitor_THT:C_Rect_L7.2mm_W2.5mm_P5.00mm_FKS2_FKP2_MKS2_MKP2
- C27: renamed from C23; value 47u -> 10u; footprint (none) -> Capacitor_THT:CP_Radial_D4.0mm_P2.00mm
- C28: renamed from C1; value 1U -> 1u; footprint (none) -> Capacitor_THT:C_Rect_L7.2mm_W4.5mm_P5.00mm_FKS2_FKP2_MKS2_MKP2
- C29: renamed from C3; footprint (none) -> Capacitor_THT:C_Rect_L7.2mm_W2.5mm_P5.00mm_FKS2_FKP2_MKS2_MKP2
- D13: renamed from D1; value D -> 1N4007; footprint (none) -> Diode_THT:D_DO-15_P10.16mm_Horizontal
- Q10: renamed from Q8; footprint Package_TO_SOT_THT:TO-126-3_Vertical -> TerminalBlock_Phoenix:TerminalBlock_Phoenix_MKDS-1,5-3_1x03_P5.00mm_Horizontal; now left out of the parts list
- Q5: renamed from Q7; footprint Package_TO_SOT_THT:TO-126-3_Vertical -> TerminalBlock_Phoenix:TerminalBlock_Phoenix_MKDS-1,5-3_1x03_P5.00mm_Horizontal; now left out of the parts list
- Q6: renamed from Q9; footprint Package_TO_SOT_THT:TO-247-3_Vertical -> TerminalBlock_Phoenix:TerminalBlock_Phoenix_MKDS-1,5-3_1x03_P5.00mm_Horizontal; now left out of the parts list
- Q7: renamed from Q6; footprint Package_TO_SOT_THT:TO-126-3_Vertical -> TerminalBlock_Phoenix:TerminalBlock_Phoenix_MKDS-1,5-3_1x03_P5.00mm_Horizontal; now left out of the parts list
- Q8: renamed from Q1; now not fitted
- Q9: renamed from Q10; footprint Package_TO_SOT_THT:TO-247-3_Vertical -> TerminalBlock_Phoenix:TerminalBlock_Phoenix_MKDS-1,5-3_1x03_P5.00mm_Horizontal; now left out of the parts list
- R28: renamed from R4; footprint (none) -> Resistor_THT:R_Axial_DIN0207_L6.3mm_D2.5mm_P10.16mm_Horizontal
- R29: renamed from R3; footprint (none) -> Resistor_THT:R_Axial_DIN0207_L6.3mm_D2.5mm_P10.16mm_Horizontal
- R30: renamed from R20; footprint (none) -> Resistor_THT:R_Axial_DIN0207_L6.3mm_D2.5mm_P10.16mm_Horizontal
- R31: renamed from R10; value R -> DNP; footprint (none) -> Resistor_THT:R_Axial_DIN0207_L6.3mm_D2.5mm_P10.16mm_Horizontal
- R32: renamed from R7; footprint (none) -> Resistor_THT:R_Axial_DIN0207_L6.3mm_D2.5mm_P10.16mm_Horizontal
- R33: renamed from R9; footprint (none) -> Resistor_THT:R_Axial_DIN0207_L6.3mm_D2.5mm_P10.16mm_Horizontal
- R34: renamed from R12; footprint (none) -> Resistor_THT:R_Axial_DIN0207_L6.3mm_D2.5mm_P10.16mm_Horizontal
- R35: renamed from R49; value R -> 470; footprint (none) -> Resistor_THT:R_Axial_DIN0207_L6.3mm_D2.5mm_P10.16mm_Horizontal
- R36: renamed from R15; footprint (none) -> Resistor_THT:R_Axial_DIN0516_L15.5mm_D5.0mm_P20.32mm_Horizontal
- R37: renamed from R8; value 150 -> 82; footprint (none) -> Resistor_THT:R_Axial_DIN0207_L6.3mm_D2.5mm_P10.16mm_Horizontal
- R38: renamed from R14; footprint (none) -> Resistor_THT:R_Axial_DIN0207_L6.3mm_D2.5mm_P10.16mm_Horizontal
- R39: renamed from R16; footprint (none) -> Resistor_THT:R_Axial_DIN0516_L15.5mm_D5.0mm_P20.32mm_Horizontal
- R40: renamed from R11; value R -> DNP; footprint (none) -> Resistor_THT:R_Axial_DIN0207_L6.3mm_D2.5mm_P10.16mm_Horizontal
- R41: renamed from R1; value R -> 0R; footprint (none) -> Resistor_THT:R_Axial_DIN0207_L6.3mm_D2.5mm_P10.16mm_Horizontal
- R43: renamed from R17; value 900 2W -> 1k 2W; footprint (none) -> Resistor_THT:R_Axial_DIN0411_L9.9mm_D3.6mm_P15.24mm_Horizontal
- R44: renamed from R50; value R -> 82; footprint (none) -> Resistor_THT:R_Axial_DIN0207_L6.3mm_D2.5mm_P10.16mm_Horizontal
- R46: renamed from R13; footprint (none) -> Resistor_THT:R_Axial_DIN0207_L6.3mm_D2.5mm_P10.16mm_Horizontal
- R47: renamed from R2; footprint (none) -> Resistor_THT:R_Axial_DIN0207_L6.3mm_D2.5mm_P10.16mm_Horizontal; now not fitted
- R48: renamed from R18; value 100 -> 150; footprint (none) -> Resistor_THT:R_Axial_DIN0207_L6.3mm_D2.5mm_P10.16mm_Horizontal
- R49: renamed from R21; footprint (none) -> Resistor_THT:R_Axial_DIN0207_L6.3mm_D2.5mm_P10.16mm_Horizontal
- R50: renamed from R6; footprint (none) -> Resistor_THT:R_Axial_DIN0207_L6.3mm_D2.5mm_P10.16mm_Horizontal
- R51: renamed from R5; footprint (none) -> Resistor_THT:R_Axial_DIN0207_L6.3mm_D2.5mm_P10.16mm_Horizontal
- R52: renamed from R19; footprint (none) -> Resistor_THT:R_Axial_DIN0207_L6.3mm_D2.5mm_P10.16mm_Horizontal
- RV3: value R_Potentiometer_Trim -> 100; footprint (none) -> Potentiometer_THT:Potentiometer_Bourns_3296W_Vertical
- RV4: renamed from RV1; footprint (none) -> Potentiometer_THT:Potentiometer_Bourns_3296W_Vertical
- RV5: renamed from RV2; now left out of the parts list
- TP13: renamed from TP14; footprint (none) -> Connector_Pin:Pin_D1.2mm_L11.3mm_W3.0mm_Flat
- TP14: renamed from TP13; footprint (none) -> Connector_Pin:Pin_D1.2mm_L11.3mm_W3.0mm_Flat
- renumbered Q4 to Q11, Q5 to Q12, Q2 to Q3, Q3 to Q4, U1 to U6
Connections:
- net +30V: now also Q3.1 (E), Q5.2 (C), Q6.2 (C), R28.1, R30.2, RV5.1, U6.7 (V+), C24.1, C26.1, D11.1 (K), J3.2 (Pin_2), J4.2 (Pin_2), J8.1 (Pin_1); no longer RV5.3
- net -30V: now also Q10.2 (C), Q12.1 (E), Q9.2 (C), R49.2, R51.2, RV5.3, U6.1 (V-), U6.4 (V-), U6.5 (V-), C31.1, C32.1, D12.2 (A), J6.2 (Pin_2), J7.2 (Pin_2), J8.3 (Pin_3); no longer RV5.1
- net GND: now also C24.2, C26.2, C30.2, C31.2, C32.2, J14.2 (Pin_2), R53.2
- net NFB: now also C34.1
- net NPN1_E: now reaches C25.2, C28.1, Q5.1 (E), Q6.1 (B), R38.1
- net NPN1_E: now also J3.3 (Pin_3), J4.3 (Pin_3)
- net NPN1_B: now reaches Q5.3 (B), R34.2
- net NPN1_B: now also J3.1 (Pin_1)
- net OFFSET_2: now reaches R52.1, RV5.2
- net OFFSET_2: now also J8.2 (Pin_2)
- net NPN3_C: now reaches Q7.2 (C), R33.2, R34.1
- net NPN3_C: now also J5.2 (Pin_2)
- net NPN3_E: now reaches C27.2, D13.2 (A), Q11.2 (C), Q7.1 (E), Q8.1 (E), R46.1, R47.2, RV4.2, RV4.3
- net NPN3_E: now also J5.3 (Pin_3), R45.1
- net NPN3_B: now reaches Q7.3 (B), R32.2, R37.1
- net NPN3_B: now also J5.1 (Pin_1)
- net PNP1_E: now reaches C28.2, C29.2, Q10.1 (E), Q9.1 (B), R38.2
- net PNP1_E: now also J6.3 (Pin_3), J7.3 (Pin_3)
- net PNP2_E: now reaches R39.2
- net PNP2_E: now also Q9.3 (E), J6.1 (Pin_1); no longer Q9.2 (C)
- net PNP1_B: now reaches Q10.3 (B), R46.2
- net PNP1_B: now also J7.1 (Pin_1)
- net at Q8.3 (B), R41.2: now also R45.2
- net NPN2_E: now reaches Q6.3 (E), R36.1
- net NPN2_E: now also J4.1 (Pin_1)
- net at R41.1, U6.6: now also C34.2
- net FLAG: now reaches U6.8 (Flag)
- net FLAG: now also R53.1
- net OUTPUT renamed OUT
- net OUT: now also D11.2 (A), D12.1 (K), R42.1; no longer R43.1
- new net: C30.1, R42.2
- new net FEEDBACK: J14.1 (Pin_1), R43.1
Other:
- note added: "Attenuator L_{min} = 1/11 L_{max} = 1/6"
- note added: "DC OFFSET TRIM POT (REAR PANEL)"
- note added: "FEEDBACK POINT AT THE OUTPUT TERMINAL"
- note added: "Gain = 1 + (1k/150) = 7.67"
- note added: "OPA552 THERMAL SHUTDOWN SOURCES 120uA WHEN DIE EXCEEDS 160°C"
- note added: "TRANSISTORS ON EXTERNAL HEATSINK"
- moved on the sheet: C25, C27, C28, C29, D13, Q10, Q11, Q12, Q3, Q4, Q5, Q6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
