File: PCB/Amplifier/Amplifier/power.kicad_sch (KiCad schematic)
At the start: 19 parts, among them J1 Screw_Terminal_01x03, U2 L7812, U3 L7912

Commit message: Worked on "amplifier" schematic
Parts:
- added TP1, TP2, TP3, TP4: TestPoint, Connector_Pin:Pin_D0.7mm_L6.5mm_W1.8mm_FlatFork, symbol Connector:TestPoint
- R24, R25: value R -> 1k
Connections:
- net +12V: now also TP3.1
- net +30V: now also TP1.1
- net -12V: now also TP4.1
- net -30V: now also TP2.1
Other:
- title: (none) -> Power

Commit message: Big commit after a long time :)
Parts:
- removed C12, C13, C6, C7: C, symbol Device:C
- added C4, C8: 10u, Capacitor_THT:CP_Radial_D4.0mm_P2.00mm, symbol Device:C_Polarized
- added H1: GND, MountingHole:MountingHole_4.3mm_M4_Pad, symbol Mechanical:MountingHole_Pad
- C1: renamed from C4; footprint (none) -> Capacitor_THT:CP_Radial_D16.0mm_P7.50mm
- C2: renamed from C8; value C -> DNP; footprint (none) -> Capacitor_THT:C_Disc_D4.3mm_W1.9mm_P5.00mm; now not fitted
- C3: renamed from C10; value C -> 1u; footprint (none) -> Capacitor_THT:C_Rect_L7.2mm_W4.5mm_P5.00mm_FKS2_FKP2_MKS2_MKP2
- C5: footprint (none) -> Capacitor_THT:CP_Radial_D16.0mm_P7.50mm
- C6: renamed from C9; value C -> DNP; footprint (none) -> Capacitor_THT:C_Disc_D4.3mm_W1.9mm_P5.00mm; now not fitted
- C7: renamed from C11; value C -> 1u; footprint (none) -> Capacitor_THT:C_Rect_L7.2mm_W4.5mm_P5.00mm_FKS2_FKP2_MKS2_MKP2
- D1: renamed from D2; value LED -> 3mm green
- D2: renamed from D3; value LED -> 3mm green
- J1: footprint (none) -> TerminalBlock_Phoenix:TerminalBlock_Phoenix_MKDS-1,5-3_1x03_P5.00mm_Horizontal
- R1: renamed from R24; footprint (none) -> Resistor_THT:R_Axial_DIN0207_L6.3mm_D2.5mm_P10.16mm_Horizontal
- R2: renamed from R22; value 1k -> 1k 2W; footprint (none) -> Resistor_THT:R_Axial_DIN0411_L9.9mm_D3.6mm_P15.24mm_Horizontal
- R3: renamed from R23; value 1k -> 1k 2W; footprint (none) -> Resistor_THT:R_Axial_DIN0411_L9.9mm_D3.6mm_P15.24mm_Horizontal
- R4: renamed from R25; footprint (none) -> Resistor_THT:R_Axial_DIN0207_L6.3mm_D2.5mm_P10.16mm_Horizontal
- TP1, TP4: footprint Connector_Pin:Pin_D0.7mm_L6.5mm_W1.8mm_FlatFork -> Connector_Pin:Pin_D1.2mm_L11.3mm_W3.0mm_Flat
- TP2: renamed from TP3; footprint Connector_Pin:Pin_D0.7mm_L6.5mm_W1.8mm_FlatFork -> Connector_Pin:Pin_D1.2mm_L11.3mm_W3.0mm_Flat
- TP3: renamed from TP2; footprint Connector_Pin:Pin_D0.7mm_L6.5mm_W1.8mm_FlatFork -> Connector_Pin:Pin_D1.2mm_L11.3mm_W3.0mm_Flat
- U1: renamed from U2; footprint (none) -> Package_TO_SOT_THT:TO-220-3_Vertical
- U2: renamed from U3; footprint (none) -> Package_TO_SOT_THT:TO-220-3_Vertical
Connections:
- net +12V: now also C4.1
- net +30V: now also J1.1 (Pin_1); no longer J1.3 (Pin_3)
- net -12V: now also C8.2
- net -30V: now also J1.3 (Pin_3); no longer J1.1 (Pin_1)
- net GND: now also C4.2, C8.1, H1.1
Other:
- moved on the sheet: C1, C3, C5, C7, D1, D2, J1, R1, R2, R3, R4, TP1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
